File: ratty.sch (EAGLE design)
At the start: 59 parts, among them IC2 L293DD, Q1 BS170, Q2 BS170, Q3 BS170, Q5 BS170, U1 ITG-32001:1

Commit message: Changed labels according to what brandon said
Parts:
- removed U$17: SPLITTER, splitter:SPLITTER
Connections:
- net C10 renamed CAP_C10_VDD_ON_MCU
- net C11 renamed CAP_C11_VDD_ON_MCU
- net C16 renamed CAP_C16_VDD_ON_MCU
- net C17 renamed CAP_C17_VBAT_ON_MCU
- net C18 renamed CAP_C18_VDD_ON_MCU
- net C19 renamed CAP_C19_VDDA/VREF_ON_MCU
- net NRST renamed NRST_CIRCUIT_MCU
- net PA_5 renamed PA_5_REC_CIRCUIT_1
- net PA_6 renamed PA_6_REC_CIRCUIT_2
- net PB_0 renamed PB_0_EMIT_CIRCUIT_3
- net PB_7 renamed PB_7_I2C1SDA_FOR_GYRO
- net PC_0 renamed PC_0_REC_CIRCUIT_3
- net PC_1 renamed PC_1_REC_CIRCUIT_4
- net PC_10 renamed PC_10_EMIT_CIRCUIT_1
- net PC_11 renamed PC_11_EMIT_CIRCUIT_2
- new net N$16: U1.AD0
- new net PB7: U1.SDA
- new net PB8_I2C1SCL_FOR_GYRO: U$4.PB8-TIM4_CH3/TIM10_CH1/I2C1_SCL/SPI5_MOSI/I2C3_SDA, U1.SCL
- net GND: now also U1.CLKIN
Changed lines of the file:
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@@
 <part name="C23" library="rcl" deviceset="C-EU" device="C0603" value="2.2nF"/>
 <part name="GND15" library="supply1" deviceset="GND" device=""/>
-<part name="U$17" library="splitter" deviceset="SPLITTER" device=""/>
+<part name="GND16" library="SparkFun" deviceset="GND" device=""/>
 </parts>
 <sheets>
@@
 <instance part="RESETBUTTON" gate="G$1" x="-20.32" y="287.02" rot="R180"/>
 <instance part="GND10" gate="1" x="208.28" y="137.16"/>
-<instance part="GND11" gate="1" x="203.2" y="147.32" rot="R270"/>
+<instance part="GND11" gate="1" x="195.58" y="147.32" rot="R270"/>
 <instance part="C20" gate="G$1" x="281.94" y="147.32"/>
 <instance part="C21" gate="G$1" x="297.18" y="147.32"/>
@@
 <instance part="C23" gate="G$1" x="332.74" y="147.32"/>
 <instance part="GND15" gate="1" x="332.74" y="132.08"/>
-<instance part="U$17" gate="G$1" x="269.24" y="177.8"/>
+<instance part="GND16" gate="1" x="254" y="144.78" rot="R90"/>
 </instances>
 <busses>
@@
 <segment>
 <pinref part="U1" gate="G$1" pin="RESV-G"/>
-<wire x1="218.44" y1="147.32" x2="205.74" y2="147.32" width="0.1524" layer="91"/>
+<wire x1="218.44" y1="147.32" x2="198.12" y2="147.32" width="0.1524" layer="91"/>
 <pinref part="GND11" gate="1" pin="GND"/>
 </segment>
@@
 <wire x1="332.74" y1="142.24" x2="332.74" y2="134.62" width="0.1524" layer="91"/>
 <pinref part="GND15" gate="1" pin="GND"/>
+</segment>
+<segment>
+<pinref part="U1" gate="G$1" pin="CLKIN"/>
+<wire x1="246.38" y1="144.78" x2="251.46" y2="144.78" width="0.1524" layer="91"/>
+<pinref part="GND16" gate="1" pin="GND"/>
 </segment>
 </net>
@@
 </segment>
 </net>
-<net name="PB_7" class="0">
+<net name="PB_7_I2C1SDA_FOR_GYRO" class="0">
 <segment>
 <pinref part="Q5" gate="1" pin="G"/>
@@
 <wire x1="525.78" y1="215.9" x2="515.62" y2="215.9" width="0.1524" layer="91"/>
 <wire x1="515.62" y1="215.9" x2="515.62" y2="213.36" width="0.1524" layer="91"/>
-<wire x1="515.62" y1="215.9" x2="502.92" y2="215.9" width="0.1524" layer="91"/>
-<junction x="515.62" y="215.9"/>
-<label x="502.92" y="215.9" size="1.778" layer="95" rot="R180" xref="yes"/>
 </segment>
 <segment>
@@
 </segment>
 </net>
-<net name="PC_1" class="0">
+<net name="PC_1_REC_CIRCUIT_4" class="0">
 <segment>
 <pinref part="U$13" gate="G$1" pin="E"/>
@@
 </segment>
 </net>
-<net name="PA_5" class="0">
+<net name="PA_5_REC_CIRCUIT_1" class="0">
 <segment>
 <pinref part="U$6" gate="G$1" pin="E"/>
@@
 </segment>
 </net>
-<net name="PC_0" class="0">
+<net name="PC_0_REC_CIRCUIT_3" class="0">
 <segment>
 <pinref part="U$11" gate="G$1" pin="E"/>
@@
 </segment>
 </net>
-<net name="PC_10" class="0">
+<net name="PC_10_EMIT_CIRCUIT_1" class="0">
 <segment>
 <pinref part="Q1" gate="1" pin="G"/>
@@
 </segment>
 </net>
-<net name="PC_11" class="0">
+<net name="PC_11_EMIT_CIRCUIT_2" class="0">
 <segment>
 <pinref part="Q2" gate="1" pin="G"/>
@@
 </segment>
 </net>
-<net name="PB_0" class="0">
-<segment>
-<pinref part="Q3" gate="1" pin="G"/>
-<pinref part="R13" gate="G$1" pin="2"/>
-<wire x1="434.34" y1="215.9" x2="424.18" y2="215.9" width="0.1524" layer="91"/>
-<wire x1="424.18" y1="215.9" x2="424.18" y2="213.36" width="0.1524" layer="91"/>
-<wire x1="424.18" y1="215.9" x2="411.48" y2="215.9" width="0.1524" layer="91"/>
-<junction x="424.18" y="215.9"/>
-<label x="411.48" y="215.9" size="1.778" layer="95" rot="R180" xref="yes"/>
-</segment>
+<net name="PB_0_IR_CIRCUIT_3" class="0">
 <segment>
 <wire x1="203.2" y1="284.48" x2="213.36" y2="284.48" width="0.1524" layer="91"/>
@@
 </segment>
 </net>
-<net name="PA_6" class="0">
+<net name="PA_6_REC_CIRCUIT_2" class="0">
 <segment>
 <pinref part="U$9" gate="G$1" pin="E"/>
@@
 </segment>
 </net>
-<net name="C17" class="0">
+<net name="CAP_C17_VBAT_ON_MCU" class="0">
 <segment>
 <pinref part="C17" gate="G$1" pin="2"/>
@@
 </segment>
 </net>
-<net name="C10" class="0">
+<net name="CAP_C10_VDD_ON_MCU" class="0">
 <segment>
 <wire x1="60.96" y1="317.5" x2="53.34" y2="317.5" width="0.1524" layer="91"/>
@@
 </segment>
 </net>
-<net name="C11" class="0">
+<net name="CAP_C11_VDD_ON_MCU" class="0">
 <segment>
 <wire x1="60.96" y1="314.96" x2="53.34" y2="314.96" width="0.1524" layer="91"/>
@@
 </segment>
 </net>
-<net name="C16" class="0">
+<net name="CAP_C16_VDD_ON_MCU" class="0">
 <segment>
 <wire x1="60.96" y1="312.42" x2="53.34" y2="312.42" width="0.1524" layer="91"/>
@@
 </segment>
 </net>
-<net name="C18" class="0">
+<net name="CAP_C18_VDD_ON_MCU" class="0">
 <segment>
 <wire x1="60.96" y1="309.88" x2="53.34" y2="309.88" width="0.1524" layer="91"/>
@@
 </segment>
 </net>
-<net name="C19" class="0">
+<net name="CAP_C19_VDDA/VREF_ON_MCU" class="0">
 <segment>
 <wire x1="60.96" y1="307.34" x2="53.34" y2="307.34" width="0.1524" layer="91"/>
@@
 </segment>
 </net>
-<net name="NRST" class="0">
+<net name="NRST_CIRCUIT_MCU" class="0">
 <segment>
 <pinref part="U$4" gate="G$1" pin="NRST"/>
@@
 </segment>
 </net>
+<net name="PB7" class="0">
+<segment>
+<pinref part="U1" gate="G$1" pin="SDA"/>
+<wire x1="246.38" y1="160.02" x2="251.46" y2="160.02" width="0.1524" layer="91"/>
+<label x="251.46" y="160.02" size="1.778" layer="95" xref="yes"/>
+</segment>
+</net>
+<net name="N$16" class="0">
+<segment>
+<pinref part="U1" gate="G$1" pin="AD0"/>
+<wire x1="246.38" y1="147.32" x2="251.46" y2="147.32" width="0.1524" layer="91"/>
+</segment>
+</net>
+<net name="PB8_I2C1SCL_FOR_GYRO" class="0">
+<segment>
+<pinref part="U$4" gate="G$1" pin="PB8-TIM4_CH3/TIM10_CH1/I2C1_SCL/SPI5_MOSI/I2C3_SDA"/>
+<wire x1="203.2" y1="264.16" x2="205.74" y2="264.16" width="0.1524" layer="91"/>
+<label x="205.74" y="264.16" size="1.778" layer="95" xref="yes"/>
+</segment>
+<segment>
+<pinref part="U1" gate="G$1" pin="SCL"/>
+<wire x1="246.38" y1="157.48" x2="251.46" y2="157.48" width="0.1524" layer="91"/>
+<label x="251.46" y="157.48" size="1.778" layer="95" xref="yes"/>
+</segment>
+</net>
+<net name="PB_0_EMIT_CIRCUIT_3" class="0">
+<segment>
+<pinref part="Q3" gate="1" pin="G"/>
+<pinref part="R13" gate="G$1" pin="2"/>
+<wire x1="434.34" y1="215.9" x2="424.18" y2="215.9" width="0.1524" layer="91"/>
+<wire x1="424.18" y1="215.9" x2="424.18" y2="213.36" width="0.1524" layer="91"/>
+<wire x1="424.18" y1="215.9" x2="411.48" y2="215.9" width="0.1524" layer="91"/>
+<junction x="424.18" y="215.9"/>
+<label x="411.48" y="215.9" size="1.778" layer="95" rot="R180" xref="yes"/>
+</segment>
+</net>

Commit message: finished gyro according to Aravinds advice
Connections:
- removed net N$16: U1.AD0
- removed net PB7: U1.SDA
- removed net PB_7_I2C1SDA_FOR_GYRO: Q5.G, R15.2
- new net PB7_I2CSDA_FOR_GYRO: U$4.PB7-TIM4_CH2/I2C1_SDA/USART1_RX/SDIO_D0, U1.SDA
- new net PB9_GYROCLK: U$4.PB9-TIM4_CH4/TIM11_CH11/I2C1_SDA/SPI2_NSS/I2C2_SDA, U1.CLKIN
- new net PB_1_EMIT_CIRCUIT_4: Q5.G, R15.2, U$4.PB1-TIM1_CH3N/TIM3_CH4/SPI5_NSS
- net GND: now also U1.AD0, U1.INT; no longer U1.CLKIN
Other:
- moved on the sheet: C12, C13, C14, C15, C20, C21, C22, C23, C6, C7, C8, C9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
