File: ratty.brd (EAGLE design)
At the start: 616 x 652 mm, 87 parts, among them IC2 L293DD, Q1 MOSFET-NCHANNELBSS123LT1G, Q2 MOSFET-NCHANNELBSS123LT1G, Q3 MOSFET-NCHANNELBSS123LT1G, Q5 MOSFET-NCHANNELBSS123LT1G, U1 ITG-32001:1

Commit message: I need to pay attention in cs 111
Routing:
- net NRST_CIRCUIT_MCU: track 22.0 -> 60.1 mm, vias 0 -> 2
- net 3.3V: track 85.3 -> 100.6 mm, vias 4 -> 6
- net RED_LED: track 0.00 -> 8.82 mm, vias 0 -> 2
Changed lines of the file:
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@@
 <wire x1="70.993" y1="41.275" x2="65.2644" y2="41.275" width="0.508" layer="1"/>
 <wire x1="65.2644" y1="41.275" x2="64.5786" y2="41.9608" width="0.508" layer="1"/>
+<wire x1="34.303078125" y1="34.969671875" x2="33.6296" y2="33.6042" width="0.3048" layer="1"/>
+<via x="33.6296" y="33.6042" extent="1-16" drill="0.6"/>
+<wire x1="33.6296" y1="33.6042" x2="33.0708" y2="34.163" width="0.3048" layer="16"/>
+<wire x1="33.0708" y1="34.163" x2="33.0708" y2="36.4744" width="0.508" layer="16"/>
+<via x="33.0708" y="36.4744" extent="1-16" drill="0.6"/>
+<wire x1="33.0708" y1="36.4744" x2="33.492196875" y2="36.895796875" width="0.3048" layer="1"/>
+<wire x1="33.492196875" y1="36.895796875" x2="33.492196875" y2="37.605478125" width="0.3048" layer="1"/>
+<wire x1="34.303078125" y1="34.969671875" x2="35.0012" y2="36.195" width="0.3048" layer="1"/>
+<wire x1="35.0012" y1="36.195" x2="35.941" y2="36.6014" width="0.508" layer="1"/>
+<wire x1="35.941" y1="36.6014" x2="39.497" y2="34.7472" width="0.508" layer="1"/>
+<wire x1="39.605671875" y1="32.16209375" x2="39.624" y2="32.1564" width="0.3048" layer="1"/>
+<wire x1="39.624" y1="32.1564" x2="40.259" y2="33.4264" width="0.3048" layer="1"/>
+<wire x1="40.259" y1="33.4264" x2="39.497" y2="34.7472" width="0.508" layer="1"/>
+<wire x1="40.21351875" y1="47.6820125" x2="47.5606" y2="71.0184" width="0" layer="19" extent="1-1"/>
+<wire x1="39.637478125" y1="45.0446" x2="40.21351875" y2="47.6820125" width="0" layer="19" extent="1-1"/>
+<wire x1="35.941" y1="36.6014" x2="39.637478125" y2="45.0446" width="0" layer="19" extent="1-1"/>
+<wire x1="44.03505625" y1="33.15484375" x2="40.259" y2="33.4264" width="0" layer="19" extent="1-1"/>
 <wire x1="48.373921875" y1="32.65254375" x2="44.03505625" y2="33.15484375" width="0" layer="19" extent="1-1"/>
-<wire x1="34.303078125" y1="34.969671875" x2="39.605671875" y2="32.16209375" width="0" layer="19" extent="1-1"/>
-<wire x1="33.0839875" y1="37.19726875" x2="34.303078125" y2="34.969671875" width="0" layer="19" extent="1-1"/>
-<wire x1="39.637478125" y1="45.0446" x2="47.0766" y2="39.0691875" width="0" layer="19" extent="1-1"/>
+<wire x1="47.0766" y1="38.89931875" x2="48.373921875" y2="32.65254375" width="0" layer="19" extent="1-1"/>
 <wire x1="52.0328" y1="17.7038" x2="48.373921875" y2="32.65254375" width="0" layer="19" extent="1-1"/>
+<wire x1="51.601" y1="11.6586" x2="52.0328" y2="17.7038" width="0" layer="19" extent="1-1"/>
+<wire x1="51.6128" y1="8.4954" x2="51.601" y2="11.6586" width="0" layer="19" extent="1-1"/>
+<wire x1="58.3834" y1="15.0354" x2="52.0328" y2="17.7038" width="0" layer="19" extent="1-1"/>
+<wire x1="61.4036" y1="12.5984" x2="58.3834" y2="15.0354" width="0" layer="19" extent="1-1"/>
+<wire x1="64.5786" y1="41.9608" x2="48.207225" y2="40.1998125" width="0" layer="19" extent="1-1"/>
 </signal>
 <signal name="TO_C5_CAP">
@@
 <wire x1="63.6016" y1="3.8354" x2="63.6016" y2="5.1034" width="0.3048" layer="1"/>
 <wire x1="63.6016" y1="5.1034" x2="63.7158" y2="5.2176" width="0.3048" layer="1"/>
-<wire x1="45.8606" y1="3.5052" x2="36.954375" y2="33.56588125" width="0" layer="19" extent="1-1"/>
+<wire x1="36.954375" y1="33.56588125" x2="36.4236" y2="32.512" width="0.3048" layer="1"/>
+<wire x1="34.9504" y1="29.464" x2="46.9646" y2="17.4498" width="0.3048" layer="16"/>
+<via x="46.9646" y="17.4498" extent="1-16" drill="0.6"/>
+<wire x1="46.9646" y1="17.4498" x2="47.0662" y2="17.4498" width="0.3048" layer="1"/>
+<wire x1="47.0662" y1="17.4498" x2="47.6504" y2="16.8656" width="0.3048" layer="1"/>
+<wire x1="47.6504" y1="16.8656" x2="47.6504" y2="15.0368" width="0.3048" layer="1"/>
+<wire x1="47.6504" y1="15.0368" x2="45.1104" y2="12.4968" width="0.3048" layer="1"/>
+<wire x1="45.1104" y1="12.4968" x2="45.1104" y2="4.2554" width="0.3048" layer="1"/>
+<wire x1="45.1104" y1="4.2554" x2="45.8606" y2="3.5052" width="0.3048" layer="1"/>
+<wire x1="36.4236" y1="32.512" x2="35.5346" y2="32.512" width="0.3048" layer="1"/>
+<wire x1="35.5346" y1="32.512" x2="34.8488" y2="31.9532" width="0.3048" layer="1"/>
+<via x="34.8488" y="31.9532" extent="1-16" drill="0.6"/>
+<wire x1="34.8488" y1="31.9532" x2="34.9504" y2="29.464" width="0.3048" layer="16"/>
 </signal>
 <signal name="GYROVLOGIC">
@@
 <contactref element="U$4" pad="8"/>
 <contactref element="R9" pad="1"/>
-<wire x1="40.3234" y1="26.8986" x2="37.39625625" y2="33.331915625" width="0" layer="19" extent="1-1"/>
+<wire x1="37.39625625" y1="33.331915625" x2="36.6522" y2="31.9532" width="0.3048" layer="1"/>
+<wire x1="36.6522" y1="31.9532" x2="36.0172" y2="31.7246" width="0.3048" layer="1"/>
+<via x="36.0172" y="31.7246" extent="1-16" drill="0.6"/>
+<wire x1="36.0172" y1="31.7246" x2="36.1696" y2="31.3436" width="0.3048" layer="16"/>
+<wire x1="36.1696" y1="31.3436" x2="39.2176" y2="28.2956" width="0.3048" layer="16"/>
+<via x="39.2176" y="28.2956" extent="1-16" drill="0.6"/>
+<wire x1="39.2176" y1="28.2956" x2="39.2176" y2="28.0044" width="0.3048" layer="1"/>
+<wire x1="39.2176" y1="28.0044" x2="40.3234" y2="26.8986" width="0.3048" layer="1"/>
 </signal>
 <signal name="BLUE_LED">

Commit message: Did one side of MCU
Parts:
- moved R9 0.05 mm to (41.2, 26.9)
Routing:
- net ENCODER2_1: track 0.00 -> 16.5 mm, vias 0 -> 1
- net ENCODER2_2: track 0.00 -> 16.0 mm, vias 0 -> 3
- net GREEN_LED: track 0.00 -> 15.4 mm, vias 0 -> 2
- net BLUE_LED: track 0.00 -> 14.9 mm, vias 0 -> 2
- net VOLTAGE_BATTERY_1: track 0.00 -> 9.20 mm

Commit message: More routing
Parts:
- moved C18 1.18 mm to (46.8, 31.5)
Routing:
- net DGND: track 179.6 -> 262.6 mm, vias 16 -> 20
- net 5V: track 150.1 -> 226.2 mm, vias 5 -> 7
- net 3.3V: track 100.9 -> 162.1 mm, vias 6 -> 11
- net PC9_REC_CIRCUIT_4: track 0.00 -> 56.2 mm, vias 0 -> 4
- net DIP_BUTTON_1: track 0.00 -> 48.3 mm, vias 0 -> 4
- net PC_11_EMIT_CIRCUIT_2: track 5.39 -> 52.3 mm, vias 0 -> 4
- net PC6_TX_PIN: track 0.00 -> 25.1 mm, vias 0 -> 2
- net PC7_RX_PIN: track 0.00 -> 23.1 mm, vias 0 -> 1
- net N$14: track 0.00 -> 19.9 mm, vias 0 -> 2
- net DIP_BUTTON_4: track 0.00 -> 16.5 mm, vias 0 -> 2
- net DIP_BUTTON_3: track 0.00 -> 16.4 mm, vias 0 -> 2
- net DIP_BUTTON_2: track 0.00 -> 14.5 mm, vias 0 -> 2
- net GND: track 89.9 -> 94.9 mm
- net N$13: track 0.00 -> 2.69 mm
- net ENCODER1_2: track 31.2 -> 29.5 mm
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
Commit message: More routing
Routing:
- net N$13: track 2.69 -> 14.3 mm, vias 0 -> 2
Changed lines of the file:
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@@
 <wire x1="39.7256" y1="46.0756" x2="39.7256" y2="47.19409375" width="0.508" layer="1"/>
 <wire x1="39.7256" y1="47.19409375" x2="40.21351875" y2="47.6820125" width="0.508" layer="1"/>
-<wire x1="39.96573125" y1="47.9298" x2="47.5606" y2="71.0184" width="0" layer="19" extent="1-1"/>
 <wire x1="64.5786" y1="41.9608" x2="48.6156" y2="38.8112" width="0" layer="19" extent="1-1"/>
+<wire x1="47.5606" y1="71.0184" x2="39.96573125" y2="47.9298" width="0" layer="19" extent="1-1"/>
 </signal>
 <signal name="TO_C5_CAP">
@@
 <wire x1="41.0718" y1="45.5676" x2="42.2148" y2="45.7708" width="0.3048" layer="1"/>
 <wire x1="42.2148" y1="45.7708" x2="42.5196" y2="46.0248" width="0.3048" layer="1"/>
-<wire x1="42.5196" y1="46.0248" x2="44.5262" y2="52.6288" width="0" layer="19" extent="1-1"/>
+<wire x1="42.5196" y1="46.0248" x2="42.926" y2="46.7106" width="0.3048" layer="1"/>
+<via x="42.926" y="46.7106" extent="1-16" drill="0.4064"/>
+<wire x1="42.926" y1="46.7106" x2="42.8752" y2="49.8856" width="0.3048" layer="16"/>
+<wire x1="42.8752" y1="49.8856" x2="41.3512" y2="51.4096" width="0.3048" layer="16"/>
+<wire x1="41.3512" y1="51.4096" x2="41.3512" y2="52.0192" width="0.3048" layer="16"/>
+<wire x1="41.3512" y1="52.0192" x2="41.0972" y2="52.2732" width="0.3048" layer="16"/>
+<wire x1="41.0972" y1="52.2732" x2="41.0972" y2="52.9082" width="0.3048" layer="16"/>
+<wire x1="41.0972" y1="52.9082" x2="41.1988" y2="53.0098" width="0.3048" layer="16"/>
+<via x="41.1988" y="53.0098" extent="1-16" drill="0.4064"/>
+<wire x1="41.1988" y1="53.0098" x2="41.4782" y2="53.2892" width="0.3048" layer="1"/>
+<wire x1="41.4782" y1="53.2892" x2="43.4086" y2="53.2892" width="0.3048" layer="1"/>
+<wire x1="43.4086" y1="53.2892" x2="44.069" y2="52.6288" width="0.3048" layer="1"/>
+<wire x1="44.069" y1="52.6288" x2="44.5262" y2="52.6288" width="0.3048" layer="1"/>
 </signal>
 <signal name="N$14">
@@
 <wire x1="57.6326" y1="42.8244" x2="51.8414" y2="42.8244" width="0.508" layer="1"/>
 <wire x1="51.8414" y1="42.8244" x2="48.5902" y2="46.0756" width="0.508" layer="1"/>
-<wire x1="48.5902" y1="46.0756" x2="43.9928" y2="46.0756" width="0.508" layer="1"/>
+<wire x1="48.5902" y1="46.0756" x2="44.0182" y2="46.0756" width="0.508" layer="1"/>
 <wire x1="66.9192125" y1="38.156203125" x2="66.3194" y2="38.7604" width="0.3048" layer="1"/>
 <wire x1="66.3194" y1="38.7604" x2="65.121215625" y2="39.9542" width="0.508" layer="1"/>
 <wire x1="42.73065625" y1="43.40684375" x2="43.3578" y2="44.6024" width="0.3048" layer="1"/>
-<wire x1="43.9928" y1="46.0756" x2="43.3578" y2="44.6024" width="0.508" layer="1"/>
+<wire x1="44.0182" y1="46.0756" x2="43.3578" y2="44.6024" width="0.508" layer="1"/>
 </signal>
 <signal name="GYROCLK">
@@
 <contactref element="U1" pad="1"/>
 <wire x1="42.288775" y1="43.640809375" x2="42.7482" y2="44.577" width="0.3048" layer="1"/>
-<wire x1="42.7482" y1="44.577" x2="42.5958" y2="44.9072" width="0.3048" layer="1"/>
-<wire x1="42.5958" y1="44.9072" x2="43.5356" y2="46.7614" width="0.3048" layer="1"/>
-<wire x1="43.5356" y1="46.7614" x2="48.7934" y2="46.7614" width="0.3048" layer="1"/>
-<wire x1="48.7934" y1="46.7614" x2="52.0446" y2="43.5102" width="0.3048" layer="1"/>
+<wire x1="42.7482" y1="44.577" x2="42.7228" y2="44.9072" width="0.3048" layer="1"/>
+<wire x1="42.7228" y1="44.9072" x2="43.7134" y2="46.7106" width="0.3048" layer="1"/>
+<wire x1="43.7134" y1="46.7106" x2="48.7934" y2="46.6852" width="0.3048" layer="1"/>
+<wire x1="48.7934" y1="46.6852" x2="52.0446" y2="43.5102" width="0.3048" layer="1"/>
 <wire x1="52.0446" y1="43.5102" x2="57.9628" y2="43.5102" width="0.3048" layer="1"/>
 <wire x1="57.9628" y1="43.5102" x2="60.0456" y2="41.4274" width="0.3048" layer="1"/>

Commit message: Down to 29 airwires boiiis
Routing:
- net PC8_REC_CIRCUIT_3: track 0.00 -> 53.8 mm, vias 0 -> 2
- net 3.3V: track 162.1 -> 193.2 mm, vias 11 -> 15
- net DIP_BUTTON_4: track 16.5 -> 37.2 mm, vias 2 -> 4
- net DGND: track 262.6 -> 282.1 mm, vias 20 -> 22
- net VOLTAGE_BATTERY_2: track 0.00 -> 13.2 mm, vias 0 -> 2
- net TO_R18/C25: track 0.00 -> 12.0 mm, vias 0 -> 2
- net 5V: track 226.2 -> 235.8 mm, vias 7 -> 8
- net TO_Q3_MOS: track 0.00 -> 6.86 mm
- net PA_6_REC_CIRCUIT_2: track 5.49 -> 6.15 mm
- net N$20: track 14.2 -> 14.8 mm
