File: ratty.brd (EAGLE design)
At the start: 616 x 652 mm, 87 parts, among them IC2 L293DD, Q1 MOSFET-NCHANNELBSS123LT1G, Q2 MOSFET-NCHANNELBSS123LT1G, Q3 MOSFET-NCHANNELBSS123LT1G, Q5 MOSFET-NCHANNELBSS123LT1G, U1 ITG-32001:1

Commit message: Routed some more
Routing:
- net PA_6_REC_CIRCUIT_2: track 6.15 -> 63.9 mm, vias 0 -> 4
- net PC_10_EMIT_CIRCUIT_1: track 4.06 -> 58.0 mm, vias 0 -> 4
- net PC9_REC_CIRCUIT_4: track 56.2 -> 95.1 mm, vias 4 -> 9
- net PB_1_EMIT_CIRCUIT_4: track 5.41 -> 31.7 mm, vias 0 -> 2
- net PA_7_REC_CIRCUIT_1: track 0.00 -> 22.8 mm, vias 0 -> 2
- net TO_R19/C28: track 14.4 -> 36.8 mm, vias 2 -> 4
- net N$19: track 0.00 -> 21.2 mm, vias 0 -> 4
- net TO_R18/C25: track 12.0 -> 33.1 mm, vias 2 -> 4
- net VOLTAGE_BATTERY_2: track 13.2 -> 30.4 mm, vias 2 -> 4
- net 3.3V: track 193.2 -> 209.2 mm
- net PB_0_EMIT_CIRCUIT_3: track 14.7 -> 28.7 mm
- net N$16: track 0.00 -> 8.77 mm, vias 0 -> 2
- net AGND: track 142.3 -> 147.2 mm, vias 2 -> 4
- net GYROVLOGIC: track 36.3 -> 40.6 mm, vias 2 -> 4
- net DGND: track 282.1 -> 284.9 mm

Commit message: Routed some more
Routing:
- net PC8_REC_CIRCUIT_3: track 54.1 -> 92.3 mm, vias 2 -> 6
- net DGND: track 284.9 -> 307.2 mm
- net 3.3V: track 209.2 -> 195.0 mm
- net BATTERY_1: track 79.5 -> 77.6 mm
- net PC6_TX_PIN: track 25.1 -> 26.7 mm

Commit message: Almost done
Routing:
- net 3.3V: track 195.0 -> 233.8 mm, vias 15 -> 18
- net DIP_BUTTON_2: track 14.5 -> 37.7 mm, vias 2 -> 6
- net DGND: track 307.2 -> 327.8 mm, vias 22 -> 26
- net AGND: track 147.2 -> 149.1 mm
- net TO_R18/C25: track 33.1 -> 32.5 mm

Commit message: 1 airwire left
Routing:
- net N$2: track 6.38 -> 111.8 mm, vias 0 -> 2
- net PA_7_REC_CIRCUIT_1: track 22.8 -> 98.8 mm, vias 2 -> 5
- net DGND: track 327.8 -> 358.8 mm, vias 26 -> 29
- net TO_Q5_MOS: track 0.00 -> 14.4 mm
- net VOLTAGE_BATTERY_1: track 9.20 -> 15.9 mm
- net 3.3V: track 233.8 -> 235.7 mm
- net R_DIGITAL_IN_2: track 47.3 -> 48.2 mm

Commit message: Finished
Parts:
- moved C15 0.67 mm to (3.45, 20.5), turned to 180 degrees
- moved C14 0.67 mm to (3.45, 22.5), turned to 180 degrees
Routing:
- net 5V: track 236.2 -> 240.3 mm
- net DGND: track 358.8 -> 359.7 mm
- net GND: track 94.9 -> 95.4 mm, vias 4 -> 6
Changed lines of the file:
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@@
 <?xml version="1.0" encoding="utf-8"?>
 <!DOCTYPE eagle SYSTEM "eagle.dtd">
-<eagle version="7.7.0">
+<eagle version="8.0.0">
 <drawing>
 <settings>
@@
 <attribute name="PROD_ID" value="TRANS-08345" x="69.85" y="27.7368" size="1.778" layer="27" rot="R270" display="off"/>
 </element>
-<element name="C14" library="rcl" package="C0603" value="0.1uF" x="4.1148" y="22.6314"/>
-<element name="C15" library="rcl" package="C0603" value="4.7uF" x="4.1148" y="20.574"/>
+<element name="C14" library="rcl" package="C0603" value="0.1uF" x="3.4544" y="22.5298" rot="R180"/>
+<element name="C15" library="rcl" package="C0603" value="4.7uF" x="3.4544" y="20.4724" rot="R180"/>
 <element name="U$8" library="Futura 1.0 motor mount template" package="FUTURA_V1.0_MOTOT_MOUNT" value="FUTURA_V1.0_MOTOR_MOUNT" x="-10.0076" y="37.2364" rot="R270"/>
 <element name="U1" library="SparkFun-Sensors" package="QFN-24_ITG3200_1:1" value="ITG-32001:1" x="68.9356" y="37.2364" rot="R45">
@@
 <wire x1="11.557" y1="10.3124" x2="11.7348" y2="10.4902" width="0.762" layer="1"/>
 <wire x1="7.1374" y1="14.13" x2="6.6548" y2="14.6126" width="1.524" layer="1"/>
-<wire x1="6.6548" y1="14.6126" x2="6.6548" y2="24.8784" width="1.524" layer="1"/>
 <wire x1="5.8674" y1="14.13" x2="7.1374" y2="14.13" width="1.524" layer="1"/>
-<wire x1="6.6548" y1="24.8784" x2="4.6092" y2="26.924" width="1.524" layer="1"/>
 <wire x1="4.6092" y1="26.924" x2="4.6092" y2="28.0806" width="1.524" layer="1"/>
 <wire x1="4.6092" y1="28.0806" x2="3.7592" y2="28.9306" width="1.524" layer="1"/>
@@
 <wire x1="2.9972" y1="40.7162" x2="3.2766" y2="40.4368" width="1.524" layer="16"/>
 <wire x1="3.2766" y1="40.4368" x2="3.2766" y2="39.2176" width="1.524" layer="16"/>
+<wire x1="6.6548" y1="14.6126" x2="6.6294" y2="14.6126" width="1.524" layer="1"/>
+<wire x1="6.6294" y1="14.6126" x2="6.2484" y2="18.669" width="1.524" layer="1"/>
+<via x="6.2484" y="18.669" extent="1-16" drill="1.6256"/>
+<wire x1="6.2484" y1="18.669" x2="6.2992" y2="18.796" width="1.524" layer="16"/>
+<wire x1="6.2992" y1="25.4" x2="5.9944" y2="25.2222" width="1.524" layer="16"/>
+<via x="5.9944" y="25.2222" extent="1-16" drill="1.6256"/>
+<wire x1="5.9944" y1="25.2222" x2="6.184" y2="25.3492" width="1.524" layer="1"/>
+<wire x1="6.184" y1="25.3492" x2="4.6092" y2="26.924" width="1.524" layer="1"/>
+<wire x1="6.2992" y1="18.796" x2="6.2992" y2="25.4" width="1.524" layer="16"/>
 </signal>
 <signal name="5V">
@@
 <wire x1="6.5922" y1="28.6258" x2="8.3702" y2="26.8478" width="1.524" layer="1"/>
 <wire x1="8.3702" y1="26.8478" x2="8.3702" y2="23.8506" width="1.524" layer="1"/>
-<wire x1="8.3702" y1="23.8506" x2="8.3702" y2="21.3106" width="1.524" layer="1"/>
+<wire x1="8.3702" y1="22.5298" x2="8.3702" y2="21.3106" width="1.524" layer="1"/>
+<wire x1="8.3702" y1="22.5298" x2="8.3702" y2="23.8506" width="1.524" layer="1"/>
 <wire x1="8.3702" y1="21.3106" x2="8.3448" y2="19.177" width="1.524" layer="1"/>
 <wire x1="8.3448" y1="19.177" x2="8.3956" y2="19.1262" width="1.524" layer="1"/>
@@
 <wire x1="12.065" y1="53.721" x2="11.3792" y2="53.0352" width="1.524" layer="16"/>
 <wire x1="11.3792" y1="53.0352" x2="11.3792" y2="47.5488" width="1.524" layer="16"/>
-<wire x1="3.2648" y1="20.574" x2="3.2648" y2="22.6314" width="1.524" layer="1"/>
 <wire x1="3.3274" y1="8.73" x2="4.5974" y2="8.73" width="1.524" layer="1"/>
 <wire x1="5.3632" y1="6.8682" x2="4.5822" y2="6.8682" width="0.762" layer="1"/>
@@
 <wire x1="76.466534375" y1="42.545" x2="74.93" y2="41.008465625" width="1.524" layer="16"/>
 <wire x1="76.466534375" y1="42.545" x2="73.4314" y2="42.545" width="1.524" layer="16"/>
-<wire x1="8.3702" y1="21.3106" x2="3.2648" y2="20.574" width="0" layer="19" extent="1-1"/>
+<wire x1="4.3044" y1="20.4724" x2="4.3044" y2="22.5298" width="1.524" layer="1"/>
+<wire x1="4.3044" y1="22.5298" x2="8.3702" y2="22.5298" width="1.524" layer="1"/>
 </signal>
 <signal name="BATTERY_1">
@@
 <wire x1="2.3114" y1="10.6426" x2="2.3114" y2="11.3284" width="1.524" layer="1"/>
 <via x="2.3114" y="11.3284" extent="1-16" drill="1.6256"/>
-<wire x1="2.3114" y1="11.3284" x2="2.3114" y2="15.875" width="1.524" layer="16"/>
-<wire x1="2.3114" y1="15.875" x2="1.8288" y2="16.3576" width="1.524" layer="16"/>
-<wire x1="1.8288" y1="16.3576" x2="1.8288" y2="23.6728" width="1.524" layer="16"/>
+<wire x1="2.3114" y1="11.3284" x2="1.8288" y2="15.5702" width="1.524" layer="16"/>
+<wire x1="1.8288" y1="15.5702" x2="1.8288" y2="23.6728" width="1.524" layer="16"/>
 <wire x1="2.9092" y1="24.7532" x2="2.9092" y2="24.8548" width="1.524" layer="16"/>
 <wire x1="2.9092" y1="24.8548" x2="2.921" y2="24.8666" width="1.524" layer="16"/>
@@
 <wire x1="12.3444" y1="20.2692" x2="12.2174" y2="20.3962" width="0.3048" layer="1"/>
 <wire x1="41.726878125" y1="46.907584375" x2="41.726878125" y2="46.883078125" width="0.3048" layer="1"/>
-<wire x1="4.9648" y1="20.574" x2="4.9648" y2="22.6314" width="1.524" layer="1"/>
+<wire x1="2.6044" y1="22.5298" x2="2.6044" y2="20.4724" width="1.524" layer="1"/>
 <wire x1="19.3548" y1="21.0566" x2="18.5674" y2="20.2692" width="0.508" layer="16"/>
-<wire x1="4.8514" y1="16.6116" x2="9.017" y2="16.6116" width="1.524" layer="16"/>
-<via x="9.017" y="16.6116" extent="1-16" drill="1.6256"/>
-<wire x1="9.017" y1="16.6116" x2="10.0956" y2="17.6902" width="1.524" layer="1"/>
+<wire x1="4.6736" y1="16.1544" x2="9.652" y2="16.51" width="1.524" layer="16"/>
+<via x="9.652" y="16.51" extent="1-16" drill="1.6256"/>
+<wire x1="9.652" y1="16.51" x2="10.0956" y2="17.6902" width="1.524" layer="1"/>
 <wire x1="10.0956" y1="17.6902" x2="10.0956" y2="19.1262" width="1.524" layer="1"/>
-<wire x1="4.8514" y1="16.6116" x2="4.3688" y2="17.0942" width="1.524" layer="16"/>
-<via x="4.3688" y="17.0942" extent="1-16" drill="1.6256"/>
-<wire x1="4.3688" y1="17.0942" x2="4.3688" y2="18.4658" width="1.524" layer="1"/>
-<wire x1="4.3688" y1="18.4658" x2="4.9784" y2="19.0754" width="1.524" layer="1"/>
-<wire x1="4.9784" y1="19.0754" x2="4.9784" y2="20.5604" width="1.524" layer="1"/>
-<wire x1="4.9784" y1="20.5604" x2="4.9648" y2="20.574" width="1.524" layer="1"/>
+<wire x1="4.6736" y1="16.1544" x2="4.0132" y2="16.8656" width="1.524" layer="16"/>
+<via x="4.0132" y="16.8656" extent="1-16" drill="1.6256"/>
+<wire x1="3.7338" y1="18.161" x2="4.0132" y2="16.8656" width="1.524" layer="1"/>
 <wire x1="58.2262" y1="71.3334" x2="58.2262" y2="72.4314" width="0.4064" layer="1"/>
 <wire x1="58.2262" y1="72.4314" x2="58.166" y2="72.4916" width="0.4064" layer="1"/>
@@
 <wire x1="39.1414" y1="36.83" x2="34.8234" y2="36.83" width="0.3048" layer="1"/>
 <wire x1="11.9126" y1="17.6022" x2="10.0076" y2="17.6022" width="0.508" layer="16"/>
-<wire x1="10.0076" y1="17.6022" x2="9.017" y2="16.6116" width="0.508" layer="16"/>
+<wire x1="10.0076" y1="17.6022" x2="9.652" y2="16.51" width="0.508" layer="16"/>
+<wire x1="2.6044" y1="20.4724" x2="2.6044" y2="19.7984" width="1.524" layer="1"/>
+<wire x1="2.6044" y1="19.7984" x2="3.7338" y2="18.161" width="1.524" layer="1"/>
 </signal>
 <signal name="N$2">

Commit message: Beginning to work on fixing up the mouse
Parts:
- removed C4: 10 uF, rcl:C0603
Connections:
- removed net TO_C4_CAP: C4.2, U$5.OUT
- new net REC_CIRCUIT_3: R4.2, U$11.E, U$4.24
- new net REC_CIRCUIT_4: R12.2, U$13.E, U$4.25
- net 3.3V: now also U$5.OUT; no longer C4.1, IC2.20
- net 5V: now also IC2.20
- net AGND: no longer U1.11, U1.12, U1.18, U1.9
- net DGND: now also U1.11, U1.12, U1.18, U1.9
- net PA_6_REC_CIRCUIT_2: no longer U$4.22
- net PA_7_REC_CIRCUIT_1: no longer U$4.23
- net PC8_REC_CIRCUIT_3: no longer R4.2, U$11.E
- net PC9_REC_CIRCUIT_4: no longer R12.2, U$13.E
Routing:
- net PC8_REC_CIRCUIT_3: track 92.3 -> 37.1 mm, vias 6 -> 4
- net REC_CIRCUIT_3: track 0.00 -> 54.1 mm, vias 0 -> 2
- net AGND: track 149.1 -> 142.5 mm
- net DGND: track 359.7 -> 363.4 mm
- net PC9_REC_CIRCUIT_4: track 95.7 -> 92.5 mm
- net TO_C4_CAP: track 2.70 -> 0.00 mm
- net 3.3V: track 235.7 -> 238.3 mm
- net PA_6_REC_CIRCUIT_2: track 64.0 -> 62.9 mm
- net PA_7_REC_CIRCUIT_1: track 98.8 -> 97.7 mm

Commit message: Ripped left side up
Parts:
- added R30, R31: 10k, rcl:R0603
Connections:
- net 3.3V: now also R30.2, R31.2
- net I2CSCL_FOR_GYRO: now also R31.1
- net I2CSDA_FOR_GYRO: now also R30.1
Routing:
- net 5V: track 240.3 -> 118.1 mm, vias 8 -> 4
- net GND: track 95.4 -> 10.1 mm, vias 6 -> 1
- net BATTERY_2: track 91.4 -> 12.1 mm, vias 2 -> 0
- net 3.3V: track 238.3 -> 171.8 mm, vias 18 -> 14
- net BATTERY_1: track 77.6 -> 20.1 mm, vias 4 -> 0
- net DGND: track 363.4 -> 327.3 mm, vias 29 -> 25
- net TO_C5_CAP: track 21.4 -> 0.00 mm, vias 2 -> 0

Commit message: Changed IR and changing LED
Parts:
- removed R16, R17: 120, rcl:R0603
- R9: value 120 -> (none)
- moved R9 369.5 mm to (-298.7, -117.8)
Connections:
- net REC_CIRCUIT_3 renamed PC4_REC_CIRCUIT_3
- net REC_CIRCUIT_4 renamed PC5_REC_CIRCUIT_4
- removed net N$18: R9.2, U$17.R
- removed net N$19: R16.2, U$17.B
- removed net N$20: R17.2, U$17.G
- removed net PC8_REC_CIRCUIT_3: U$4.39
- removed net PC9_REC_CIRCUIT_4: U$4.53
- removed net PC_10_EMIT_CIRCUIT_1: Q1.1, R6.2, U$4.51
- removed net PC_11_EMIT_CIRCUIT_2: Q2.1, R10.2, U$4.52
- new net N$1: R9.1, U$17.A
- new net PB13_EMIT_CIRCUIT_1: Q1.1, R6.2, U$4.34
- new net PB14_EMIT_CIRCUIT_2: Q2.1, R10.2, U$4.35
- net 3.3V: no longer U$17.A
- net 5V: now also R9.2
- net BLUE_LED: now also U$17.B; no longer R16.1
- net DIP_BUTTON_2: now also U$4.29; no longer U$4.35
- net DIP_BUTTON_3: now also U$4.62; no longer U$4.34
- net GREEN_LED: now also U$17.G; no longer R17.1
- net PA_6_REC_CIRCUIT_2: now also U$4.22
- net PA_7_REC_CIRCUIT_1: now also U$4.23
- net RED_LED: now also U$17.R; no longer R9.1
Routing:
- net PC9_REC_CIRCUIT_4: track 92.5 -> 0.00 mm, vias 9 -> 0
- net PC_10_EMIT_CIRCUIT_1: track 58.0 -> 0.00 mm, vias 4 -> 0
- net PB13_EMIT_CIRCUIT_1: track 0.00 -> 56.8 mm, vias 0 -> 4
- net PC_11_EMIT_CIRCUIT_2: track 52.3 -> 0.00 mm, vias 4 -> 0
- net PB14_EMIT_CIRCUIT_2: track 0.00 -> 51.3 mm, vias 0 -> 4
- net PC8_REC_CIRCUIT_3: track 37.1 -> 0.00 mm, vias 4 -> 0
- net N$18: track 23.3 -> 0.00 mm, vias 2 -> 0
- net N$19: track 21.2 -> 0.00 mm, vias 4 -> 0
- net N$20: track 14.8 -> 0.00 mm, vias 2 -> 0
- net GREEN_LED: track 15.3 -> 13.7 mm
- net DIP_BUTTON_3: track 16.4 -> 14.9 mm
- net DIP_BUTTON_2: track 37.7 -> 36.3 mm
- net RED_LED: track 9.56 -> 8.32 mm
