File: encoder.brd (EAGLE design)
At the start: 31.8 x 34.3 mm, 5 parts

Commit message: I guess we're done
Parts:
- moved C1 1.31 mm to (7.87, 30.6)
- moved JP2 1.31 mm to (26.8, 5.71)
- moved JP1 1.31 mm to (2.67, 5.59)
- moved C2 1.31 mm to (7.75, 26.4)
- moved U$1 1.31 mm to (14.9, 28.4)
Other:
- board size 31.8 x 34.3 mm -> 29.7 x 34.3 mm
Changed lines of the file:
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@@
 <?xml version="1.0" encoding="utf-8"?>
 <!DOCTYPE eagle SYSTEM "eagle.dtd">
-<eagle version="7.7.0">
+<eagle version="8.0.0">
 <drawing>
 <settings>
@@
 <board>
 <plain>
-<text x="3.81" y="10.16" size="1.4224" layer="21" rot="R180">5V</text>
-<text x="10.795" y="3.81" size="1.4224" layer="21" rot="R180">GND</text>
-<text x="6.985" y="3.81" size="1.4224" layer="22" rot="MR180">GND</text>
-<text x="1.905" y="10.16" size="1.4224" layer="22" rot="MR180">5V</text>
-<text x="6.604" y="28.956" size="1.27" layer="22" rot="MR270">0.1uF</text>
-<text x="6.858" y="24.765" size="1.27" layer="21" rot="R90">0.1uF</text>
-<text x="8.001" y="20.701" size="1.27" layer="21">10uF</text>
-<text x="11.43" y="20.701" size="1.27" layer="22" rot="MR0">10uF</text>
-<text x="27.305" y="8.89" size="1.4224" layer="21">B</text>
-<text x="28.575" y="8.89" size="1.4224" layer="22" rot="MR0">B</text>
-<text x="29.845" y="3.81" size="1.4224" layer="22" rot="MR180">A</text>
-<text x="31.115" y="3.81" size="1.4224" layer="21" rot="R180">A</text>
-<wire x1="0" y1="34.29" x2="31.75" y2="34.29" width="0.4064" layer="20"/>
-<wire x1="31.75" y1="34.29" x2="31.75" y2="0" width="0.4064" layer="20"/>
-<wire x1="31.75" y1="0" x2="21.717" y2="0" width="0.4064" layer="20"/>
-<wire x1="21.717" y1="0" x2="21.717" y2="22.606" width="0.4064" layer="20"/>
-<wire x1="21.717" y1="22.606" x2="10.668" y2="22.606" width="0.4064" layer="20"/>
-<wire x1="10.668" y1="22.606" x2="10.668" y2="0" width="0.4064" layer="20"/>
-<wire x1="10.668" y1="0" x2="0" y2="0" width="0.4064" layer="20"/>
+<text x="2.667" y="9.525" size="1.4224" layer="21" rot="R180">5V</text>
+<text x="9.652" y="3.175" size="1.4224" layer="21" rot="R180">GND</text>
+<text x="5.842" y="3.175" size="1.4224" layer="22" rot="MR180">GND</text>
+<text x="0.762" y="9.525" size="1.4224" layer="22" rot="MR180">5V</text>
+<text x="5.461" y="28.321" size="1.27" layer="22" rot="MR270">0.1uF</text>
+<text x="5.715" y="24.13" size="1.27" layer="21" rot="R90">0.1uF</text>
+<text x="6.858" y="20.066" size="1.27" layer="21">10uF</text>
+<text x="10.287" y="20.066" size="1.27" layer="22" rot="MR0">10uF</text>
+<text x="26.162" y="8.255" size="1.4224" layer="21">B</text>
+<text x="27.432" y="8.255" size="1.4224" layer="22" rot="MR0">B</text>
+<text x="28.702" y="3.175" size="1.4224" layer="22" rot="MR180">A</text>
+<text x="29.972" y="3.175" size="1.4224" layer="21" rot="R180">A</text>
+<wire x1="0" y1="34.29" x2="29.718" y2="34.29" width="0.4064" layer="20"/>
+<wire x1="29.718" y1="34.29" x2="29.718" y2="0.127" width="0.4064" layer="20"/>
+<wire x1="29.718" y1="0.127" x2="21.717" y2="0.127" width="0.4064" layer="20"/>
+<wire x1="21.717" y1="0.127" x2="21.717" y2="21.844" width="0.4064" layer="20"/>
+<wire x1="21.717" y1="21.844" x2="7.874" y2="21.717" width="0.4064" layer="20"/>
+<wire x1="7.874" y1="21.717" x2="7.874" y2="0" width="0.4064" layer="20"/>
+<wire x1="7.874" y1="0" x2="0" y2="0" width="0.4064" layer="20"/>
 <wire x1="0" y1="0" x2="0" y2="34.29" width="0.4064" layer="20"/>
 </plain>
@@
 </autorouter>
 <elements>
-<element name="C1" library="rcl" package="C0603" value="0.1uF" x="9.017" y="31.242"/>
-<element name="C2" library="rcl" package="C0603" value="10uF" x="8.89" y="27.051"/>
-<element name="U$1" library="AS5304_AS5306-Encoder" package="AS5304/AS5306-ENCODER" value="AS5304/AS5306-ENCODER" x="16.002" y="29.083"/>
-<element name="JP1" library="SparkFun" package="1X02_LOCK" value="" x="3.81" y="6.223"/>
-<element name="JP2" library="SparkFun" package="1X02_LOCK" value="" x="27.9527" y="6.35" rot="R180"/>
+<element name="C1" library="rcl" package="C0603" value="0.1uF" x="7.874" y="30.607"/>
+<element name="C2" library="rcl" package="C0603" value="10uF" x="7.747" y="26.416"/>
+<element name="U$1" library="AS5304_AS5306-Encoder" package="AS5304/AS5306-ENCODER" value="AS5304/AS5306-ENCODER" x="14.859" y="28.448"/>
+<element name="JP1" library="SparkFun" package="1X02_LOCK" value="" x="2.667" y="5.588"/>
+<element name="JP2" library="SparkFun" package="1X02_LOCK" value="" x="26.8097" y="5.715" rot="R180"/>
 </elements>
 <signals>
@@
 <polygon width="0.4064" layer="16">
 <vertex x="0" y="34.29"/>
-<vertex x="31.75" y="34.29"/>
-<vertex x="31.75" y="0"/>
-<vertex x="21.717" y="0"/>
-<vertex x="21.717" y="22.606"/>
-<vertex x="10.668" y="22.606"/>
-<vertex x="10.668" y="0"/>
+<vertex x="30.48" y="34.29"/>
+<vertex x="30.48" y="0"/>
+<vertex x="22.606" y="0.127"/>
+<vertex x="22.098" y="21.971"/>
+<vertex x="8.382" y="21.717"/>
+<vertex x="8.128" y="0"/>
 <vertex x="0" y="0"/>
 </polygon>
-<wire x1="9.867" y1="31.242" x2="12.561" y2="31.242" width="0.4064" layer="1"/>
-<wire x1="12.561" y1="31.242" x2="13.102" y2="31.783" width="0.4064" layer="1"/>
-<wire x1="13.102" y1="31.783" x2="13.102" y2="30.84" width="0.4064" layer="1"/>
-<wire x1="13.102" y1="30.84" x2="13.589" y2="30.353" width="0.4064" layer="1"/>
-<wire x1="13.589" y1="30.353" x2="15.7226" y2="30.353" width="0.4064" layer="1"/>
-<wire x1="15.7226" y1="30.353" x2="16.3576" y2="30.988" width="0.4064" layer="1"/>
-<wire x1="16.3576" y1="30.988" x2="16.3576" y2="31.7774" width="0.4064" layer="1"/>
-<wire x1="16.3576" y1="31.7774" x2="16.352" y2="31.783" width="0.4064" layer="1"/>
-<wire x1="9.74" y1="27.051" x2="9.74" y2="31.115" width="0.4064" layer="1"/>
-<wire x1="9.74" y1="31.115" x2="9.867" y2="31.242" width="0.4064" layer="1"/>
-<wire x1="9.74" y1="27.051" x2="12.434" y2="27.051" width="0.4064" layer="1"/>
-<wire x1="12.434" y1="27.051" x2="13.102" y2="26.383" width="0.4064" layer="1"/>
-<wire x1="9.74" y1="27.051" x2="9.74" y2="25.996" width="0.4064" layer="1"/>
-<wire x1="9.74" y1="25.996" x2="7.747" y2="24.003" width="0.4064" layer="1"/>
-<wire x1="7.747" y1="24.003" x2="7.747" y2="7.4422" width="0.4064" layer="1"/>
-<wire x1="7.747" y1="7.4422" x2="6.5278" y2="6.223" width="0.4064" layer="1"/>
+<wire x1="8.724" y1="30.607" x2="11.418" y2="30.607" width="0.4064" layer="1"/>
+<wire x1="11.418" y1="30.607" x2="11.959" y2="31.148" width="0.4064" layer="1"/>
+<wire x1="11.959" y1="31.148" x2="11.959" y2="30.205" width="0.4064" layer="1"/>
+<wire x1="11.959" y1="30.205" x2="12.446" y2="29.718" width="0.4064" layer="1"/>
+<wire x1="12.446" y1="29.718" x2="14.5796" y2="29.718" width="0.4064" layer="1"/>
+<wire x1="14.5796" y1="29.718" x2="15.2146" y2="30.353" width="0.4064" layer="1"/>
+<wire x1="15.2146" y1="30.353" x2="15.2146" y2="31.1424" width="0.4064" layer="1"/>
+<wire x1="15.2146" y1="31.1424" x2="15.209" y2="31.148" width="0.4064" layer="1"/>
+<wire x1="8.597" y1="26.416" x2="8.597" y2="30.48" width="0.4064" layer="1"/>
+<wire x1="8.597" y1="30.48" x2="8.724" y2="30.607" width="0.4064" layer="1"/>
+<wire x1="8.597" y1="26.416" x2="11.291" y2="26.416" width="0.4064" layer="1"/>
+<wire x1="11.291" y1="26.416" x2="11.959" y2="25.748" width="0.4064" layer="1"/>
+<wire x1="8.597" y1="26.416" x2="8.597" y2="25.361" width="0.4064" layer="1"/>
+<wire x1="8.597" y1="25.361" x2="6.604" y2="23.368" width="0.4064" layer="1"/>
+<wire x1="6.604" y1="23.368" x2="6.604" y2="6.8072" width="0.4064" layer="1"/>
+<wire x1="6.604" y1="6.8072" x2="5.3848" y2="5.588" width="0.4064" layer="1"/>
 </signal>
 <signal name="A">
 <contactref element="U$1" pad="2_A"/>
 <contactref element="JP2" pad="2"/>
-<wire x1="13.752" y1="26.383" x2="13.752" y2="25.364" width="0.4064" layer="1"/>
-<wire x1="13.752" y1="25.364" x2="14.605" y2="24.511" width="0.4064" layer="1"/>
-<wire x1="14.605" y1="24.511" x2="22.86" y2="24.511" width="0.4064" layer="1"/>
-<wire x1="22.86" y1="24.511" x2="23.749" y2="23.622" width="0.4064" layer="1"/>
-<wire x1="23.749" y1="23.622" x2="23.749" y2="7.8359" width="0.4064" layer="1"/>
-<wire x1="23.749" y1="7.8359" x2="25.2349" y2="6.35" width="0.4064" layer="1"/>
+<wire x1="12.609" y1="25.748" x2="12.609" y2="24.729" width="0.4064" layer="1"/>
+<wire x1="12.609" y1="24.729" x2="13.462" y2="23.876" width="0.4064" layer="1"/>
+<wire x1="13.462" y1="23.876" x2="21.717" y2="23.876" width="0.4064" layer="1"/>
+<wire x1="21.717" y1="23.876" x2="22.606" y2="22.987" width="0.4064" layer="1"/>
+<wire x1="22.606" y1="22.987" x2="22.606" y2="7.2009" width="0.4064" layer="1"/>
+<wire x1="22.606" y1="7.2009" x2="24.0919" y2="5.715" width="0.4064" layer="1"/>
 </signal>
 <signal name="5V">
@@
 <polygon width="0.4064" layer="1">
 <vertex x="0" y="34.29"/>
-<vertex x="31.75" y="34.29"/>
-<vertex x="31.75" y="0"/>
-<vertex x="21.717" y="0"/>
-<vertex x="21.717" y="22.606"/>
-<vertex x="10.668" y="22.606"/>
-<vertex x="10.668" y="0"/>
+<vertex x="30.48" y="34.29"/>
+<vertex x="30.48" y="0"/>
+<vertex x="22.606" y="0.127"/>
+<vertex x="21.971" y="21.844"/>
+<vertex x="8.255" y="21.59"/>
+<vertex x="8.128" y="0"/>
 <vertex x="0" y="0"/>
 </polygon>
@@
 <contactref element="U$1" pad="4_B"/>
 <contactref element="JP2" pad="1"/>
-<wire x1="28.1305" y1="6.35" x2="28.1305" y2="26.0985" width="0.4064" layer="1"/>
-<wire x1="28.1305" y1="26.0985" x2="25.146" y2="29.083" width="0.4064" layer="1"/>
-<wire x1="25.146" y1="29.083" x2="16.2052" y2="29.083" width="0.4064" layer="1"/>
-<wire x1="16.2052" y1="29.083" x2="15.0622" y2="27.94" width="0.4064" layer="1"/>
-<wire x1="15.0622" y1="27.94" x2="15.0622" y2="26.3932" width="0.4064" layer="1"/>
-<wire x1="15.0622" y1="26.3932" x2="15.052" y2="26.383" width="0.4064" layer="1"/>
+<wire x1="26.9875" y1="5.715" x2="26.9875" y2="25.4635" width="0.4064" layer="1"/>
+<wire x1="26.9875" y1="25.4635" x2="24.003" y2="28.448" width="0.4064" layer="1"/>
+<wire x1="24.003" y1="28.448" x2="15.0622" y2="28.448" width="0.4064" layer="1"/>
+<wire x1="15.0622" y1="28.448" x2="13.9192" y2="27.305" width="0.4064" layer="1"/>
+<wire x1="13.9192" y1="27.305" x2="13.9192" y2="25.7582" width="0.4064" layer="1"/>
+<wire x1="13.9192" y1="25.7582" x2="13.909" y2="25.748" width="0.4064" layer="1"/>
 </signal>
 <signal name="INDEX">
